File: ESP32/ESP32/ESP32.kicad_sch (KiCad schematic)
At the start: 21 parts, among them J1 F_Header_Ultrasonic, J2 F_Header_Temp, Q1 SS8050-G, Q2 SS8050-G, SW1 SW_Push, SW2 SW_Push, U2 ESP32-S3-WROOM-1-N16R2

Commit message: Update Schematic
Parts:
- added MQ135: Gas Sensor, symbol Connector_Generic:Conn_01x04
- added MicroUSB_5V1A_Wall: Conn_01x05, symbol Connector_Generic:Conn_01x05
- added R10, R9: 1k, symbol Device:R
- added R11: 2.2k, symbol Device:R
- added USB_UART: Conn_01x06, symbol Connector_Generic:Conn_01x06
- renumbered J2 to DHT22, J1 to HC-SR04, U1 to ZMOD
Connections:
- net CAMERA_SDA is gone; now on net ZMOD_SDA: U2.30 (IO37)
- net GPIO15 is gone; now on net S: U2.8 (IO15)
- net GPIO5 is gone; now on net Trig: U2.5 (IO5)
- net GPIO6 is gone; now on net Echo: U2.6 (IO6)
- net +3V3: now also DHT22.1 (Pin_1)
- net +5V: now also MQ135.1 (Pin_1), MicroUSB_5V1A_Wall.1 (Pin_1); no longer DHT22.1 (Pin_1)
- net DTR: now also USB_UART.6 (Pin_6)
- net Echo: now also R10.2, R11.1; no longer HC-SR04.3 (Pin_3)
- net GND: now also MQ135.2 (Pin_2), MicroUSB_5V1A_Wall.5 (Pin_5), R11.2, USB_UART.1 (Pin_1)
- net RTS: now also USB_UART.2 (Pin_2)
- net RX: now also USB_UART.4 (Pin_4)
- net TX: now also USB_UART.5 (Pin_5)
- net ZMOD_SDA: now reaches ZMOD. (VSS)
- net CAMERA_MISO renamed ZMOD_RES_N
- net ZMOD_RES_N: now also ZMOD. (VSS)
- net CAMERA_SCK renamed ZMOD_INT
- net ZMOD_INT: now also ZMOD. (VSS)
- net CAMERA_SCL renamed ZMOD_SCL
- net ZMOD_SCL: now also ZMOD. (VSS)
- net GPIO7 renamed A0
- net A0: now also R9.1
- new net: MQ135.4 (Pin_4), R9.2
- new net: HC-SR04.3 (Pin_3), R10.1
Other:
- moved on the sheet: DHT22, HC-SR04, ZMOD
