File: ESP32/Sensor Board/ESP32.kicad_sch (KiCad schematic)
At the start: 27 parts, among them Q1 SS8050-G, Q2 SS8050-G, SW1 SW_Push, SW2 SW_Push, U2 ESP32-S3-WROOM-1-N16R2

Commit message: Added voltage regulators to both schematics
Parts:
- added C5: 10u, symbol Device:C
- added U1: AZ1117-3.3, symbol Regulator_Linear:AZ1117-3.3
Connections:
- net +5V: now also C5.1, U1.3 (VI)
- net GND: now also C5.2, U1.1 (GND)
- new net +3.3V: U1.2 (VO)
Changed lines of the file:
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@@
   (junction (at 177.8 44.45) (diameter 0) (color 0 0 0 0)
   )
+  (junction (at 213.36 142.24) (diameter 0) (color 0 0 0 0)
+  )
   (junction (at 64.77 76.2) (diameter 0) (color 0 0 0 0)
   )
@@
   )
   (wire (pts (xy 87.63 101.6) (xy 90.17 101.6))
+    (stroke (width 0) (type default))
+  )
+  (wire (pts (xy 208.28 142.24) (xy 213.36 142.24))
     (stroke (width 0) (type default))
   )
@@
     )
   )
+  (symbol (lib_id "Regulator_Linear:AZ1117-3.3") (at 220.98 142.24 0) (unit 1)
+    (in_bom yes) (on_board yes) (dnp no) (fields_autoplaced)
+    (property "Reference" "U1" (at 220.98 135.89 0)
+      (effects (font (size 1.27 1.27)))
+    )
+    (property "Value" "AZ1117-3.3" (at 220.98 138.43 0)
+      (effects (font (size 1.27 1.27)))
+    )
+    (property "Footprint" "" (at 220.98 135.89 0)
+      (effects (font (size 1.27 1.27) italic) hide)
+    )
+    (property "Datasheet" "https://www.diodes.com/assets/Datasheets/AZ1117.pdf" (at 220.98 142.24 0)
+      (effects (font (size 1.27 1.27)) hide)
+    )
+    (pin "1")
+    (pin "3")
+    (pin "2")
+    (instances
+      (project "ESP32"
+        (path "/668738a4-4fba-4c81-8219-00fa4ae32623"
+          (reference "U1") (unit 1)
+        )
+      )
+    )
+  )
   (symbol (lib_id "power:GND") (at 97.79 49.53 0) (unit 1)
     (in_bom yes) (on_board yes) (dnp no) (fields_autoplaced)
@@
     )
   )
+  (symbol (lib_name "GND_2") (lib_id "power:GND") (at 208.28 149.86 0) (unit 1)
+    (in_bom yes) (on_board yes) (dnp no) (fields_autoplaced)
+    (property "Reference" "#PWR027" (at 208.28 156.21 0)
+      (effects (font (size 1.27 1.27)) hide)
+    )
+    (property "Value" "GND" (at 208.28 154.94 0)
+      (effects (font (size 1.27 1.27)))
+    )
+    (property "Footprint" "" (at 208.28 149.86 0)
+      (effects (font (size 1.27 1.27)) hide)
+    )
+    (property "Datasheet" "" (at 208.28 149.86 0)
+      (effects (font (size 1.27 1.27)) hide)
+    )
+    (pin "1")
+    (instances
+      (project "ESP32"
+        (path "/668738a4-4fba-4c81-8219-00fa4ae32623"
+          (reference "#PWR027") (unit 1)
+        )
+      )
+    )
+  )
   (symbol (lib_id "power:+5V") (at 142.24 170.18 0) (unit 1)
     (in_bom yes) (on_board yes) (dnp no) (fields_autoplaced)
@@
     )
   )
+  (symbol (lib_id "power:+3.3V") (at 228.6 142.24 0) (unit 1)
+    (in_bom yes) (on_board yes) (dnp no) (fields_autoplaced)
+    (property "Reference" "#PWR025" (at 228.6 146.05 0)
+      (effects (font (size 1.27 1.27)) hide)
+    )
+    (property "Value" "+3.3V" (at 228.6 137.16 0)
+      (effects (font (size 1.27 1.27)))
+    )
+    (property "Footprint" "" (at 228.6 142.24 0)
+      (effects (font (size 1.27 1.27)) hide)
+    )
+    (property "Datasheet" "" (at 228.6 142.24 0)
+      (effects (font (size 1.27 1.27)) hide)
+    )
+    (pin "1")
+    (instances
+      (project "ESP32"
+        (path "/668738a4-4fba-4c81-8219-00fa4ae32623"
+          (reference "#PWR025") (unit 1)
+        )
+      )
+    )
+  )
+  (symbol (lib_id "Device:C") (at 208.28 146.05 0) (unit 1)
+    (in_bom yes) (on_board yes) (dnp no) (fields_autoplaced)
+    (property "Reference" "C5" (at 212.09 144.78 0)
+      (effects (font (size 1.27 1.27)) (justify left))
+    )
+    (property "Value" "10u" (at 212.09 147.32 0)
+      (effects (font (size 1.27 1.27)) (justify left))
+    )
+    (property "Footprint" "" (at 209.2452 149.86 0)
+      (effects (font (size 1.27 1.27)) hide)
+    )
+    (property "Datasheet" "~" (at 208.28 146.05 0)
+      (effects (font (size 1.27 1.27)) hide)
+    )
+    (pin "2")
+    (pin "1")
+    (instances
+      (project "ESP32"
+        (path "/668738a4-4fba-4c81-8219-00fa4ae32623"
+          (reference "C5") (unit 1)
+        )
+      )
+    )
+  )
   (symbol (lib_id "power:GND") (at 140.97 59.69 0) (unit 1)
     (in_bom yes) (on_board yes) (dnp no) (fields_autoplaced)
@@
         (path "/668738a4-4fba-4c81-8219-00fa4ae32623"
           (reference "#PWR02") (unit 1)
+        )
+      )
+    )
+  )
+  (symbol (lib_name "GND_1") (lib_id "power:GND") (at 220.98 149.86 0) (unit 1)
+    (in_bom yes) (on_board yes) (dnp no) (fields_autoplaced)
+    (property "Reference" "#PWR026" (at 220.98 156.21 0)
+      (effects (font (size 1.27 1.27)) hide)
+    )
+    (property "Value" "GND" (at 220.98 154.94 0)
+      (effects (font (size 1.27 1.27)))
+    )
+    (property "Footprint" "" (at 220.98 149.86 0)
+      (effects (font (size 1.27 1.27)) hide)
+    )
+    (property "Datasheet" "" (at 220.98 149.86 0)
+      (effects (font (size 1.27 1.27)) hide)
+    )
+    (pin "1")
+    (instances
+      (project "ESP32"
+        (path "/668738a4-4fba-4c81-8219-00fa4ae32623"
+          (reference "#PWR026") (unit 1)
         )
       )
@@
         )
       )
+    )
+  )
+  (symbol (lib_id "power:+5V") (at 213.36 142.24 0) (unit 1)
+    (in_bom yes) (on_board yes) (dnp no) (fields_autoplaced)
+    (property "Reference" "#PWR024" (at 213.36 146.05 0)
+      (effects (font (size 1.27 1.27)) hide)
+    )
+    (property "Value" "+5V" (at 213.36 137.16 0)
+      (effects (font (size 1.27 1.27)))
+    )
+    (property "Footprint" "" (at 213.36 142.24 0)
+      (effects (font (size 1.27 1.27)) hide)
+    )
+    (property "Datasheet" "" (at 213.36 142.24 0)
+      (effects (font (size 1.27 1.27)) hide)
+    )
+    (pin "1")
+    (instances
+      (project "ESP32"
+        (path "/668738a4-4fba-4c81-8219-00fa4ae32623"
+          (reference "#PWR024") (unit 1)
+        )
+      )
